File: tube_screamer.kicad_pcb (KiCad board)
At the start: 2 copper layers, 80 x 100 mm, 68 parts, among them J1 Jack_6.35, J2 Jack_6.35, J3 Conn_01x05, J4 Conn_01x05, J5 Conn_01x05, J6 Barrel_Jack_Switch, J7 Conn_01x01_Socket, J8 Conn_01x01_Socket, P1 tube_screamer_front_panel, Q1 MMBT5551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

Commit message: Rotirani pinovi audio konektora, rotirani LED prekidač pinovi.
Connections:
- SW1 pad 4: 9V -> unconnected-(SW1B-A-Pad4)
- SW1 pad 6: unconnected-(SW1B-C-Pad6) -> 9V
Routing:
- net Net-(J1-PadT): track 121.7 -> 142.8 mm
- net Net-(C11-Pad2): track 51.5 -> 70.6 mm
- net 9V: track 189.2 -> 184.2 mm, vias 6 -> 4
- net 0: vias 86 -> 84
