File: tube_screamer_front_plate/tube_screamer_front_plate.kicad_sch (KiCad schematic)
At the start: 21 parts, among them J1 top_panel_connector

Commit message: Update schematic.
Parts:
- removed H10, H9: MountingHole, MountingHole:MountingHole_3mm, symbol Mechanical:MountingHole
- removed H5, H6, H7: MountingHole_Pad, pedale:plated_pot_hole, symbol Mechanical:MountingHole_Pad
- removed JP1, JP2, JP3: SolderJumper_2_Bridged, Jumper:SolderJumper-2_P1.3mm_Bridged_RoundedPad1.0x1.5mm, symbol Jumper:SolderJumper_2_Bridged
- J1: footprint pedale:bottom_connector -> Connector_IDC:IDC-Header_2x08_P2.54mm_Vertical
Connections:
- net at J1.5 (Pin_5): now also RV2.3; no longer RV2.1
- net at J1.9 (Pin_9): now also RV2.1; no longer RV2.3
- net at RV3.1: now also J1.16 (Pin_16); no longer J1.12 (Pin_12)
- net at RV3.3: now also J1.12 (Pin_12); no longer J1.16 (Pin_16)
- net at D1.2 (A): now also J1.1 (Pin_8); no longer J1.8 (Pin_8)
- net at D2.2 (A): now also J1.3 (Pin_10); no longer J1.10 (Pin_10)
Other:
- moved on the sheet: D1, D2, RV1, RV2, RV3

Commit message: 1 Red, 3 green connector.
Parts:
- J1: footprint Connector_IDC:IDC-Header_2x08_P2.54mm_Vertical -> pedale:bottom_connector
Changed lines of the file:
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@@
 			)
 		)
-		(property "Description" ""
+		(property "Description" "Mounting Hole without connection"
 			(at 38.1 152.4 0)
 			(effects
@@
 		(pin "16"
 		)
+		(pin "3"
+		)
+		(pin "15"
+		)
+		(pin "14"
+		)
+		(pin "11"
+		)
+		(pin "13"
+		)
+		(pin "8"
+		)
+		(pin "6"
+		)
+		(pin "5"
+		)
+		(pin "2"
+		)
+		(pin "4"
+		)
+		(pin "10"
+		)
 		(pin "1"
-		)
-		(pin "15"
-		)
-		(pin "14"
-		)
-		(pin "11"
-		)
-		(pin "13"
-		)
-		(pin "8"
-		)
-		(pin "6"
-		)
-		(pin "5"
-		)
-		(pin "2"
-		)
-		(pin "4"
-		)
-		(pin "10"
-		)
-		(pin "3"
 		)
 		(pin "7"
@@
 		(pin "16"
 		)
+		(pin "3"
+		)
+		(pin "15"
+		)
+		(pin "14"
+		)
+		(pin "11"
+		)
+		(pin "13"
+		)
+		(pin "8"
+		)
+		(pin "6"
+		)
+		(pin "5"
+		)
+		(pin "2"
+		)
+		(pin "4"
+		)
+		(pin "10"
+		)
 		(pin "1"
-		)
-		(pin "15"
-		)
-		(pin "14"
-		)
-		(pin "11"
-		)
-		(pin "13"
-		)
-		(pin "8"
-		)
-		(pin "6"
-		)
-		(pin "5"
-		)
-		(pin "2"
-		)
-		(pin "4"
-		)
-		(pin "10"
-		)
-		(pin "3"
 		)
 		(pin "7"
@@
 			)
 		)
-		(property "Description" ""
+		(property "Description" "Mounting Hole without connection"
 			(at 57.15 144.78 0)
 			(effects
@@
 	)
 	(symbol
-		(lib_name "top_panel_connector_1")
 		(lib_id "pedale:top_panel_connector")
 		(at 81.28 110.49 0)
@@
 			)
 		)
-		(property "Footprint" "Connector_IDC:IDC-Header_2x08_P2.54mm_Vertical"
+		(property "Footprint" "pedale:bottom_connector"
 			(at 81.28 110.49 0)
 			(effects
@@
 		(pin "16"
 		)
+		(pin "3"
+		)
+		(pin "15"
+		)
+		(pin "14"
+		)
+		(pin "11"
+		)
+		(pin "13"
+		)
+		(pin "8"
+		)
+		(pin "6"
+		)
+		(pin "5"
+		)
+		(pin "2"
+		)
+		(pin "4"
+		)
+		(pin "10"
+		)
 		(pin "1"
-		)
-		(pin "15"
-		)
-		(pin "14"
-		)
-		(pin "11"
-		)
-		(pin "13"
-		)
-		(pin "8"
-		)
-		(pin "6"
-		)
-		(pin "5"
-		)
-		(pin "2"
-		)
-		(pin "4"
-		)
-		(pin "10"
-		)
-		(pin "3"
 		)
 		(pin "7"
@@
 			)
 		)
-		(property "Description" ""
+		(property "Description" "Mounting Hole without connection"
 			(at 38.1 144.78 0)
 			(effects
@@
 		(pin "16"
 		)
+		(pin "3"
+		)
+		(pin "15"
+		)
+		(pin "14"
+		)
+		(pin "11"
+		)
+		(pin "13"
+		)
+		(pin "8"
+		)
+		(pin "6"
+		)
+		(pin "5"
+		)
+		(pin "2"
+		)
+		(pin "4"
+		)
+		(pin "10"
+		)
 		(pin "1"
-		)
-		(pin "15"
-		)
-		(pin "14"
-		)
-		(pin "11"
-		)
-		(pin "13"
-		)
-		(pin "8"
-		)
-		(pin "6"
-		)
-		(pin "5"
-		)
-		(pin "2"
-		)
-		(pin "4"
-		)
-		(pin "10"
-		)
-		(pin "3"
 		)
 		(pin "7"
@@
 		(on_board yes)
 		(dnp no)
-		(fields_autoplaced yes)
 		(property "Reference" "D2"
 			(at 73.66 109.5374 90)
@@
 			)
 		)
-		(property "Description" ""
+		(property "Description" "Mounting Hole without connection"
 			(at 57.15 152.4 0)
 			(effects
@@
 	)
 	(symbol
-		(lib_name "top_panel_connector_2")
 		(lib_id "pedale:top_panel_connector")
 		(at 45.72 110.49 0)
@@
 			)
 		)
-		(property "Footprint" "Connector_IDC:IDC-Header_2x08_P2.54mm_Vertical"
+		(property "Footprint" "pedale:bottom_connector"
 			(at 45.72 110.49 0)
 			(effects
@@
 		(pin "16"
 		)
+		(pin "3"
+		)
+		(pin "15"
+		)
+		(pin "14"
+		)
+		(pin "11"
+		)
+		(pin "13"
+		)
+		(pin "8"
+		)
+		(pin "6"
+		)
+		(pin "5"
+		)
+		(pin "2"
+		)
+		(pin "4"
+		)
+		(pin "10"
+		)
 		(pin "1"
-		)
-		(pin "15"
-		)
-		(pin "14"
-		)
-		(pin "11"
-		)
-		(pin "13"
-		)
-		(pin "8"
-		)
-		(pin "6"
-		)
-		(pin "5"
-		)
-		(pin "2"
-		)
-		(pin "4"
-		)
-		(pin "10"
-		)
-		(pin "3"
 		)
 		(pin "7"
@@
 		(pin "16"
 		)
+		(pin "3"
+		)
+		(pin "15"
+		)
+		(pin "14"
+		)
+		(pin "11"
+		)
+		(pin "13"
+		)
+		(pin "8"
+		)
+		(pin "6"
+		)
+		(pin "5"
+		)
+		(pin "2"
+		)
+		(pin "4"
+		)
+		(pin "10"
+		)
 		(pin "1"
-		)
-		(pin "15"
-		)
-		(pin "14"
-		)
-		(pin "11"
-		)
-		(pin "13"
-		)
-		(pin "8"
-		)
-		(pin "6"
-		)
-		(pin "5"
-		)
-		(pin "2"
-		)
-		(pin "4"
-		)
-		(pin "10"
-		)
-		(pin "3"
 		)
 		(pin "7"
@@
 			)
 		)
-		(property "Description" ""
+		(property "Description" "Mounting Hole without connection"
 			(at 77.47 148.59 0)
 			(effects
@@
 		(pin "16"
 		)
+		(pin "3"
+		)
+		(pin "15"
+		)
+		(pin "14"
+		)
+		(pin "11"
+		)
+		(pin "13"
+		)
+		(pin "8"
+		)
+		(pin "6"
+		)
+		(pin "5"
+		)
+		(pin "2"
+		)
+		(pin "4"
+		)
+		(pin "10"
+		)
 		(pin "1"
 		)
-		(pin "15"
-		)
-		(pin "14"
-		)
-		(pin "11"
-		)
-		(pin "13"
-		)
-		(pin "8"
-		)
-		(pin "6"
-		)
-		(pin "5"
-		)
-		(pin "2"
-		)
-		(pin "4"
-		)
-		(pin "10"
-		)
-		(pin "3"
-		)
 		(pin "7"

Commit message: Pots checked, all good.
Connections:
- net at J1.5 (Pin_5): now also RV3.3; no longer RV2.3
- net at J1.7 (Pin_7): now also RV3.2; no longer RV2.2
- net at J1.9 (Pin_9): now also RV3.1; no longer RV2.1
- net at J1.16 (Pin_16): now also RV2.1; no longer RV3.1
- net at J1.14 (Pin_14): now also RV2.2; no longer RV3.2
- net at J1.12 (Pin_12): now also RV2.3; no longer RV3.3
- net at D1.2 (A): now also J1.8 (Pin_8); no longer J1.1 (Pin_8)
- net at D2.2 (A): now also J1.10 (1); no longer J1.3 (1)
- net at J1.2 (Pin_2): now also RV1.3; no longer RV1.1
- net at J1.6 (Pin_6): now also RV1.1; no longer RV1.3
Other:
- moved on the sheet: RV1, RV2, RV3

Commit message: Fixed diodes on front plate, fixed power schem.
Parts:
- removed JP4: SolderJumper_2_Bridged, Jumper:SolderJumper-2_P1.3mm_Bridged_RoundedPad1.0x1.5mm, symbol Jumper:SolderJumper_2_Bridged
- removed RV1, RV2, RV3: R_Potentiometer, pedale:top_plate_pot, symbol Device:R_Potentiometer
- added RV1, RV2, RV3: pot_gnd, pedale:top_plate_pot, symbol pedale:pot_gnd
Connections:
- net 0: now also H8.1, RV1.MH (2), RV2.MH (2), RV3.MH (2)
- net at J1.5 (Pin_5): now also RV3.3
- net at J1.7 (Pin_7): now also RV3.2
- net at J1.9 (Pin_9): now also RV3.1
- net at J1.16 (Pin_16): now also RV2.1
- net at J1.14 (Pin_14): now also RV2.2
- net at J1.12 (Pin_12): now also RV2.3
- net at J1.2 (Pin_2): now also RV1.3
- net at J1.4 (Pin_4): now also RV1.2
- net at J1.6 (Pin_6): now also RV1.1

Commit message: Tube screamer front plate done, library updated.
Parts:
- J1: footprint pedale:bottom_connector -> pedale:IDC-Header_2x08_faux_SMD
Changed lines of the file:
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@@
 			)
 		)
-		(property "Footprint" "pedale:bottom_connector"
+		(property "Footprint" "pedale:IDC-Header_2x08_faux_SMD"
 			(at 45.72 53.34 0)
 			(effects
@@
 			)
 		)
-		(property "Footprint" "pedale:bottom_connector"
+		(property "Footprint" "pedale:IDC-Header_2x08_faux_SMD"
 			(at 241.3 138.43 0)
 			(effects
@@
 			)
 		)
-		(property "Footprint" "pedale:bottom_connector"
+		(property "Footprint" "pedale:IDC-Header_2x08_faux_SMD"
 			(at 81.28 110.49 0)
 			(effects
@@
 			)
 		)
-		(property "Footprint" "pedale:bottom_connector"
+		(property "Footprint" "pedale:IDC-Header_2x08_faux_SMD"
 			(at 45.72 30.48 0)
 			(effects
@@
 			)
 		)
-		(property "Footprint" "pedale:bottom_connector"
+		(property "Footprint" "pedale:IDC-Header_2x08_faux_SMD"
 			(at 45.72 110.49 0)
 			(effects
@@
 			)
 		)
-		(property "Footprint" "pedale:bottom_connector"
+		(property "Footprint" "pedale:IDC-Header_2x08_faux_SMD"
 			(at 254 134.62 0)
 			(effects
@@
 			)
 		)
-		(property "Footprint" "pedale:bottom_connector"
+		(property "Footprint" "pedale:IDC-Header_2x08_faux_SMD"
 			(at 45.72 74.93 0)
 			(effects

Commit message: GND to top.
Connections:
- net 0: now also J1.3 (GND)
Changed lines of the file:
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@@
+	)
+	(symbol
+		(lib_id "Simulation_SPICE:0")
+		(at 241.3 138.43 0)
+		(unit 1)
+		(exclude_from_sim no)
+		(in_bom yes)
+		(on_board yes)
+		(dnp no)
+		(fields_autoplaced yes)
+		(property "Reference" "#GND01"
+			(at 241.3 143.51 0)
+			(effects
+				(font
+					(size 1.27 1.27)
+				)
+				(hide yes)
+			)
+		)
+		(property "Value" "0"
+			(at 241.3 135.89 0)
+			(effects
+				(font
+					(size 1.27 1.27)
+				)
+			)
+		)
+		(property "Footprint" ""
+			(at 241.3 138.43 0)
+			(effects
+				(font
+					(size 1.27 1.27)
+				)
+				(hide yes)
+			)
+		)
+		(property "Datasheet" "https://ngspice.sourceforge.io/docs/ngspice-html-manual/manual.xhtml#subsec_Circuit_elements__device"
+			(at 241.3 148.59 0)
+			(effects
+				(font
+					(size 1.27 1.27)
+				)
+				(hide yes)
+			)
+		)
+		(property "Description" "0V reference potential for simulation"
+			(at 241.3 146.05 0)
+			(effects
+				(font
+					(size 1.27 1.27)
+				)
+				(hide yes)
+			)
+		)
+		(pin "1"
+		)
+		(instances
+			(project ""
+				(path "/1fda0e48-ac05-4486-b24b-352a2425b266"
+					(reference "#GND01")
+					(unit 1)
+				)
+			)
+		)
 	)
 	(symbol
