File: tube_screamer/tube_screamer.kicad_sch (KiCad schematic)
At the start: 67 parts, among them J1 Jack_6.35, J2 Jack_6.35, J6 Barrel_Jack_Switch, J7 Conn_01x01_Socket, J8 Conn_01x01_Socket, J9 top_panel_connector, P1 front_plate, P2 bottom_plate, Q1 MMBT5551, Q10 AO3401A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

Commit message: Updated libraries.
Parts:
- SW1: footprint pedale:foot_switch_tht_and_floating -> pedale:foot_switch_tht_no_pad
Changed lines of the file:
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@@
 			)
 		)
-		(property "Footprint" "pedale:foot_switch_tht_and_floating"
+		(property "Footprint" "pedale:foot_switch_tht_no_pad"
 			(at 240.03 93.98 0)
 			(effects
@@
 			)
 		)
-		(property "Footprint" "pedale:foot_switch_tht_and_floating"
+		(property "Footprint" "pedale:foot_switch_tht_no_pad"
 			(at 165.1 119.38 0)
 			(effects

Commit message: Checklist done, only layout left.
Connections:
- net 0: now also J9.3 (GND); no longer J9.10 (GND)
- net 9V: now also J9.1 (VCC); no longer J9.8 (VCC)
- net at R28.1: now also J9.8 (Pin_8); no longer J9.1 (Pin_8)
- net at R26.1: now also J9.10 (Pin_10); no longer J9.3 (1)
Changed lines of the file:
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@@
 	)
 	(symbol
+		(lib_name "0_3")
 		(lib_id "Simulation_SPICE:0")
 		(at 87.63 67.31 0)
@@
 	)
 	(symbol
+		(lib_name "MountingHole_4")
 		(lib_id "Mechanical:MountingHole")
 		(at 40.64 100.33 0)
