File: tube_screamer_bottom_plate/tube_screamer_bottom_plate.kicad_pcb (KiCad board)
At the start: 2 copper layers, 80 x 100 mm, 8 parts

Commit message: Ready for production.
Parts:
- removed the REF** at (150.4, 79.8)
Changed lines of the file:
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@@
 			(outputformat 1)
 			(mirror no)
-			(drillshape 1)
+			(drillshape 0)
 			(scaleselection 1)
-			(outputdirectory "")
+			(outputdirectory "gerbers/")
 		)
 	)
@@
 			(stroke
 				(width 0.05)
-				(type default)
-			)
-			(fill no)
-			(layer "B.CrtYd")
-		)
-		(fp_text user "${REFERENCE}"
-			(at 0 -2.5 0)
-			(unlocked yes)
-			(layer "B.Fab")
-			(effects
-				(font
-					(size 1 1)
-					(thickness 0.15)
-				)
-				(justify mirror)
-			)
-		)
-		(embedded_fonts no)
-	)
-	(footprint "pedale:TI logo"
-		(layer "B.Cu")
-		(at 150.4 79.8 180)
-		(property "Reference" "REF**"
-			(at 0 0.2 0)
-			(unlocked yes)
-			(layer "B.SilkS")
-			(hide yes)
-			(effects
-				(font
-					(size 1 1)
-					(thickness 0.1)
-				)
-				(justify mirror)
-			)
-		)
-		(property "Value" "TI logo"
-			(at 0 -1 0)
-			(unlocked yes)
-			(layer "B.Fab")
-			(effects
-				(font
-					(size 1 1)
-					(thickness 0.15)
-				)
-				(justify mirror)
-			)
-		)
-		(property "Datasheet" ""
-			(at -5.5 3.5 0)
-			(unlocked yes)
-			(layer "B.Fab")
-			(hide yes)
-			(effects
-				(font
-					(size 1 1)
-					(thickness 0.15)
-				)
-				(justify mirror)
-			)
-		)
-		(property "Description" ""
-			(at -5.5 3.5 0)
-			(unlocked yes)
-			(layer "B.Fab")
-			(hide yes)
-			(effects
-				(font
-					(size 1 1)
-					(thickness 0.15)
-				)
-				(justify mirror)
-			)
-		)
-		(attr through_hole)
-		(fp_rect
-			(start -1.6 1.6)
-			(end 1.6 1.1)
-			(stroke
-				(width 0.1)
-				(type solid)
-			)
-			(fill yes)
-			(layer "B.SilkS")
-		)
-		(fp_circle
-			(center 0 0)
-			(end 3 0)
-			(stroke
-				(width 0.5)
-				(type default)
-			)
-			(fill no)
-			(layer "B.SilkS")
-		)
-		(fp_poly
-			(pts
-				(xy 0.4 0.2) (xy 0.9 0.5) (xy 0.9 1.3) (xy 0.4 1.3)
-			)
-			(stroke
-				(width 0.1)
-				(type solid)
-			)
-			(fill yes)
-			(layer "B.SilkS")
-		)
-		(fp_poly
-			(pts
-				(xy 0.4 -1.9) (xy 0.4 -0.1) (xy 0.9 0.2) (xy 0.9 -1.9)
-			)
-			(stroke
-				(width 0.1)
-				(type solid)
-			)
-			(fill yes)
-			(layer "B.SilkS")
-		)
-		(fp_poly
-			(pts
-				(xy -0.9 -1.9) (xy -0.9 1.2) (xy -0.4 1.2) (xy -0.4 -1.9)
-			)
-			(stroke
-				(width 0.1)
-				(type solid)
-			)
-			(fill yes)
-			(layer "B.SilkS")
-		)
-		(fp_rect
-			(start -3.4 3.3)
-			(end 3.4 -3.3)
-			(stroke
-				(width 0.05)
